Commit message: feat: inicio do exercicio 1.2 atv 2

File: 02_controle_movimento/models/my_robot/model.urdf.xacro (robot description, xacro)
@@ -1,4 +1,4 @@
 <?xml version="1.0"?>
-<robot name="my_robot">
+<robot name="my_robot" xmlns:xacro="http://www.ros.org/wiki/xacro">
   <link name="chassis">
     <inertial>
@@ -99,3 +99,31 @@
     <static>false</static>
   </gazebo>
+  <!-- ros2_control - as rodas recebem comando de velocidade e informam posicao e velocidade -->
+  <ros2_control name="GazeboSystem" type="system">
+    <hardware>
+      <plugin>gazebo_ros2_control/GazeboSystem</plugin>
+    </hardware>
+    <joint name="left_wheel_hinge">
+      <command_interface name="velocity">
+        <param name="min">-10</param>
+        <param name="max">10</param>
+      </command_interface>
+      <state_interface name="position"/>
+      <state_interface name="velocity"/>
+    </joint>
+    <joint name="right_wheel_hinge">
+      <command_interface name="velocity">
+        <param name="min">-10</param>
+        <param name="max">10</param>
+      </command_interface>
+      <state_interface name="position"/>
+      <state_interface name="velocity"/>
+    </joint>
+  </ros2_control>
+  <!-- Plugin que sobe o controller_manager dentro do Gazebo -->
+  <gazebo>
+    <plugin filename="libgazebo_ros2_control.so" name="gazebo_ros2_control">
+      <parameters>$(find controle_movimento)/config/controllers.yaml</parameters>
+    </plugin>
+  </gazebo>
 </robot>

Commit message: teclado e atrito

File: 02_controle_movimento/models/my_robot/model.urdf.xacro (robot description, xacro)
@@ -77,4 +77,5 @@
     <origin xyz="0.1 0.13 0" rpy="0 1.5707 1.5707"/>
     <axis xyz="0 0 1"/>
+    <dynamics damping="0.05" friction="0.02"/>
   </joint>
   <joint name="right_wheel_hinge" type="continuous">
@@ -83,4 +84,5 @@
     <origin xyz="0.1 -0.13 0" rpy="0 1.5707 1.5707"/>
     <axis xyz="0 0 1"/>
+    <dynamics damping="0.05" friction="0.02"/>
   </joint>
   <gazebo reference="chassis">
@@ -99,5 +101,4 @@
     <static>false</static>
   </gazebo>
-  <!-- ros2_control - as rodas recebem comando de velocidade e informam posicao e velocidade -->
   <ros2_control name="GazeboSystem" type="system">
     <hardware>
@@ -105,16 +106,18 @@
     </hardware>
     <joint name="left_wheel_hinge">
-      <command_interface name="velocity">
-        <param name="min">-10</param>
-        <param name="max">10</param>
-      </command_interface>
+      <param name="vel_kp">1.0</param>
+      <param name="vel_ki">0.5</param>
+      <param name="vel_kd">0.0</param>
+      <param name="vel_max_integral_error">10</param>
+      <command_interface name="velocity_pid"/>
       <state_interface name="position"/>
       <state_interface name="velocity"/>
     </joint>
     <joint name="right_wheel_hinge">
-      <command_interface name="velocity">
-        <param name="min">-10</param>
-        <param name="max">10</param>
-      </command_interface>
+      <param name="vel_kp">1.0</param>
+      <param name="vel_ki">0.5</param>
+      <param name="vel_kd">0.0</param>
+      <param name="vel_max_integral_error">10</param>
+      <command_interface name="velocity_pid"/>
       <state_interface name="position"/>
       <state_interface name="velocity"/>
@@ -125,4 +128,7 @@
     <plugin filename="libgazebo_ros2_control.so" name="gazebo_ros2_control">
       <parameters>$(find controle_movimento)/config/controllers.yaml</parameters>
+      <ros>
+        <remapping>diff_drive_controller/odom:=odom</remapping>
+      </ros>
     </plugin>
   </gazebo>
